File: led-dimmer-boat.kicad_pcb (KiCad board)
At the start: 2 copper layers, 62 x 30 mm, 18 parts, among them J1 PWR, J2 Prog, J3 LEDSTRIP, Q1 IRLB8721PBF, Q2 IRLB8721PBF, Q4 2N3904, SW1 M2023SS1W03, U1 ATtiny13A-PU-ND, U2 LM7805S/NOPB

Commit message: Updated schematic.pdf and added board.png
Parts:
- moved C1 1.12 mm to (134.4, 108.9)
- moved C3 1.12 mm to (130.6, 82.5)
- moved J1 1.12 mm to (157.6, 105.2)
- moved Q4 1.12 mm to (111.0, 83.2)
- moved J3 1.12 mm to (105.3, 98.7)
- moved D1 1.12 mm to (152.6, 106.4)
- moved H1 1.12 mm to (104.9, 84.2)
- moved H2 1.12 mm to (104.9, 106.2)
- moved Q2 1.12 mm to (128.8, 105.4)
- moved R2 1.12 mm to (120.0, 83.2)
- moved RV1 1.12 mm to (146.0, 98.1)
- moved SW1 1.12 mm to (153.0, 100.0)
- moved U1 1.12 mm to (133.5, 89.4)
- moved U2 1.12 mm to (137.8, 99.5)
- moved C2 1.12 mm to (141.0, 109.0)
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
Commit message: Final changes for first version
Parts:
- added R3: 10K, Resistors_SMD:R_0603_HandSoldering, F.Cu at (126.9, 82.5)
- C1, C2, C3: footprint Capacitors_SMD:C_0603 -> Capacitors_SMD:C_0603_HandSoldering
- D1: footprint Diodes_SMD:D_SOD-123 -> Diodes_SMD:D_SOD-323_HandSoldering
- R1, R2: footprint Resistors_SMD:R_0603 -> Resistors_SMD:R_0603_HandSoldering
- moved D1 0.40 mm to (152.6, 106.8)
- moved C2 0.21 mm to (141.2, 108.9)
- moved C1 0.21 mm to (134.2, 109.0)
Connections:
- J2 pad 5: RESET -> (no net)
- U1 pad 1: RESET -> Net-(R3-Pad2)
Routing:
- net RESET: track 28.9 -> 0.00 mm, vias 2 -> 0
- net Net-(R3-Pad2): track 0.00 -> 9.41 mm, vias 0 -> 1
- net +5V: track 92.2 -> 95.9 mm
- net RED_DET: track 28.4 -> 29.2 mm
- net +12V: track 16.7 -> 17.3 mm
Other:
- board text added: "+12V"
- board text added: "B"
- board text added: "G"
- board text added: "GND"
- board text added: "PWR"
- board text added: "R"

Commit message: Added JST-EH connectors
Parts:
- J1: footprint Pin_Headers:Pin_Header_Straight_1x02_Pitch2.54mm -> Connectors_JST:JST_EH_B02B-EH-A_02x2.50mm_Straight
- J3: footprint Pin_Headers:Pin_Header_Straight_1x04_Pitch2.54mm -> Connectors_JST:JST_EH_B04B-EH-A_04x2.50mm_Straight
- moved SW1 0.90 mm to (153.1, 99.1)
- moved J1 0.53 mm to (157.4, 104.7), turned to 270 degrees
- turned J3 to 90 degrees
Routing:
- net +12V: track 17.3 -> 21.8 mm
- net VDD: track 90.2 -> 91.9 mm
- net RED_SEL: track 40.6 -> 39.8 mm
- net +5V: track 95.9 -> 96.6 mm
Other:
- board text removed: "+12V"
