File: led-dimmer-boat.sch (KiCad schematic (older format))
At the start: 18 parts, among them J1 PWR, J2 Prog, J3 LEDSTRIP, Q1 IRLB8721PBF, Q2 IRLB8721PBF, Q4 2N3904, SW1 M2023SS1W03, U1 ATtiny13A-PU-ND, U2 LM7805S/NOPB

Commit message: Final changes for first version
Parts:
- added R3: 10K, Resistors_SMD:R_0603_HandSoldering, symbol Device:R
- C1, C2, C3: footprint Capacitors_SMD:C_0603 -> Capacitors_SMD:C_0603_HandSoldering
- D1: footprint Diodes_SMD:D_SOD-123 -> Diodes_SMD:D_SOD-323_HandSoldering
- R1, R2: footprint Resistors_SMD:R_0603 -> Resistors_SMD:R_0603_HandSoldering
Connections:
- net +5V: now also R3.1
- net RESET: no longer U1.1 (~RESET~/PB5)
- new net: R3.2, U1.1 (~RESET~/PB5)
Changed lines of the file:
@@
 F 0 "R1" V 5218 2750 50  0000 C CNN
 F 1 "82K" V 5309 2750 50  0000 C CNN
-F 2 "Resistors_SMD:R_0603" V 5355 2750 50  0001 C CNN
+F 2 "Resistors_SMD:R_0603_HandSoldering" V 5355 2750 50  0001 C CNN
 F 3 "~" H 5425 2750 50  0001 C CNN
 	1    5425 2750
@@
 F 0 "R2" V 5993 2275 50  0000 C CNN
 F 1 "300K" V 6084 2275 50  0000 C CNN
-F 2 "Resistors_SMD:R_0603" V 6130 2275 50  0001 C CNN
+F 2 "Resistors_SMD:R_0603_HandSoldering" V 6130 2275 50  0001 C CNN
 F 3 "~" H 6200 2275 50  0001 C CNN
 	1    6200 2275
@@
 F 0 "D1" H 1750 1583 50  0000 C CNN
 F 1 "1N5400" H 1750 1674 50  0000 C CNN
-F 2 "Diodes_SMD:D_SOD-123" H 1750 1625 50  0001 C CNN
+F 2 "Diodes_SMD:D_SOD-323_HandSoldering" H 1750 1625 50  0001 C CNN
 F 3 "http://www.vishay.com/docs/88516/1n5400.pdf" H 1750 1800 50  0001 C CNN
 	1    1750 1800
@@
 F 0 "C1" H 4293 6471 50  0000 L CNN
 F 1 "0.22uF" H 4293 6380 50  0000 L CNN
-F 2 "Capacitors_SMD:C_0603" H 4213 6275 50  0001 C CNN
+F 2 "Capacitors_SMD:C_0603_HandSoldering" H 4213 6275 50  0001 C CNN
 F 3 "~" H 4175 6425 50  0001 C CNN
 	1    4175 6425
@@
 F 0 "C2" H 5340 6446 50  0000 L CNN
 F 1 "0.1uF" H 5340 6355 50  0000 L CNN
-F 2 "Capacitors_SMD:C_0603" H 5263 6250 50  0001 C CNN
+F 2 "Capacitors_SMD:C_0603_HandSoldering" H 5263 6250 50  0001 C CNN
 F 3 "~" H 5225 6400 50  0001 C CNN
 	1    5225 6400
@@
 F 0 "C3" H 8240 2046 50  0000 L CNN
 F 1 "0.1uF" H 8240 1955 50  0000 L CNN
-F 2 "Capacitors_SMD:C_0603" H 8163 1850 50  0001 C CNN
+F 2 "Capacitors_SMD:C_0603_HandSoldering" H 8163 1850 50  0001 C CNN
 F 3 "~" H 8125 2000 50  0001 C CNN
 	1    8125 2000
@@
 Wire Wire Line
 	8450 5525 8600 5525
-Text GLabel 8825 3650 2    50   Input ~ 0
-RESET
 Wire Wire Line
 	8700 3350 8825 3350
@@
 	8700 3550 8825 3550
 Wire Wire Line
-	8700 3650 8825 3650
+	8700 3650 9325 3650
 $Comp
 L MCU_Microchip_ATtiny:ATtiny13V-10SSU U1
@@
 	1    0    0    -1
 $EndComp
+$Comp
+L power:+5V #PWR0121
+U 1 1 628A2ED2
+P 9775 3650
+F 0 "#PWR0121" H 9775 3500 50  0001 C CNN
+F 1 "+5V" H 9775 3850 28  0000 C CNN
+F 2 "" H 9775 3650 50  0000 C CNN
+F 3 "" H 9775 3650 50  0000 C CNN
+	1    9775 3650
+	1    0    0    -1
+$EndComp
+$Comp
+L Device:R R3
+U 1 1 628B1FD4
+P 9475 3650
+F 0 "R3" V 9268 3650 50  0000 C CNN
+F 1 "10K" V 9359 3650 50  0000 C CNN
+F 2 "Resistors_SMD:R_0603_HandSoldering" V 9405 3650 50  0001 C CNN
+F 3 "~" H 9475 3650 50  0001 C CNN
+	1    9475 3650
+	0    1    1    0
+$EndComp
+Wire Wire Line
+	9625 3650 9775 3650
 $EndSCHEMATC

Commit message: Added JST-EH connectors
Parts:
- J1: footprint Pin_Headers:Pin_Header_Straight_1x02_Pitch2.54mm -> Connectors_JST:JST_EH_B02B-EH-A_02x2.50mm_Straight
- J3: footprint Pin_Headers:Pin_Header_Straight_1x04_Pitch2.54mm -> Connectors_JST:JST_EH_B04B-EH-A_04x2.50mm_Straight
Changed lines of the file:
@@
 F 0 "J3" H 1118 4375 50  0000 C CNN
 F 1 "LEDSTRIP" H 1118 4466 50  0000 C CNN
-F 2 "Pin_Headers:Pin_Header_Straight_1x04_Pitch2.54mm" H 1200 4800 50  0001 C CNN
+F 2 "Connectors_JST:JST_EH_B04B-EH-A_04x2.50mm_Straight" H 1200 4800 50  0001 C CNN
 F 3 "~" H 1200 4800 50  0001 C CNN
 	1    1200 4800
@@
 F 0 "J1" H 1168 1575 50  0000 C CNN
 F 1 "PWR" H 1168 1666 50  0000 C CNN
-F 2 "Pin_Headers:Pin_Header_Straight_1x02_Pitch2.54mm" H 1250 1900 50  0001 C CNN
+F 2 "Connectors_JST:JST_EH_B02B-EH-A_02x2.50mm_Straight" H 1250 1900 50  0001 C CNN
 F 3 "~" H 1250 1900 50  0001 C CNN
 	1    1250 1900
